File: design/design.kicad_pcb (KiCad board)
At the start: 2 copper layers, 176.5 x 83.2 mm, 23 parts, among them J2 Conn_01x08_Socket, SW1 SW_Push, SW10 SW_Push, SW11 SW_Push, SW12 SW_Push, SW13 SW_Push, SW2 SW_Push, SW3 SW_Push, SW4 SW_Push, SW5 SW_Push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

Commit message: KiCad work, 3D modelling case
Parts:
- added J2: Conn_01x08_Socket, Connector_PinSocket_2.54mm:PinSocket_1x08_P2.54mm_Vertical, F.Cu at (180.5, 62.0)
Routing:
- net Net-(A1-GPIO1): track 95.9 -> 101.6 mm
Other:
- board text added: "1"
- board text added: "2"
- board text added: "3"
- board text added: "4"
- board text added: "5"
- board text added: "A"
- board text added: "B"
- board text added: "X"
- board text added: "Y"
- board text added: "connect display here"
- board text added: "do not use this header"
- board text added: "help"
- board text added: "reset"
- board text added: "support for display (J2) must be 20/23rds along the length of display board to ensure support does not touch the extended black part, which would stop the display from sitting flat. (>50.5mm from the lowest part of J1)"
- board text added: "thank you hack club <3 (((o(*ﾟ▽ﾟ*)o)))"
- board text added: "←"
- board text added: "↑"
- board text added: "→"
- board text added: "↓"
