File: design/design.kicad_pcb (KiCad board)
At the start: 2 copper layers, 176.5 x 83.2 mm, 30 parts, among them J2 Conn_01x08_Socket, SW1 SW_Push, SW10 SW_Push, SW11 SW_Push, SW12 SW_Push, SW13 SW_Push, SW2 SW_Push, SW3 SW_Push, SW4 SW_Push, SW5 SW_Push, SW6 SW_Push, SW7 SW_Push, SW8 SW_Push, SW9 SW_Push, U1 MPU-6050

Commit message: Updated PCB with style
Parts:
- added G*** (x3): LOGO, LOGO, F.Cu at (203.9, 128.8)
Other:
- board text added: "PCB rev 2.1.0"
- board text added: "al"
- board text added: "designed by felix in London UK"
- board text added: "function"
- board text added: "gyroscope"
- board text added: "keyboard"
- board text added: "multi"
- board text added: "we love you soup"
- board text added: "（⊙ｏ⊙）"
- board text removed: "gyroscope （⊙ｏ⊙）"
