File: design/design.kicad_pcb (KiCad board)
At the start: 2 copper layers, 176.5 x 83.2 mm, 33 parts, among them J2 Conn_01x08_Socket, SW1 SW_Push, SW10 SW_Push, SW11 SW_Push, SW12 SW_Push, SW13 SW_Push, SW2 SW_Push, SW3 SW_Push, SW4 SW_Push, SW5 SW_Push, SW6 SW_Push, SW7 SW_Push, SW8 SW_Push, SW9 SW_Push, U1 MPU-6050

Commit message: Version using LSM6DS3 (C967633) chip
Parts:
- removed C3: 2.2nF, Capacitor_SMD:C_0603_1608Metric
- removed C4: 10nF, Capacitor_SMD:C_0603_1608Metric
- removed REF** (x4): MountingHole_3.2mm_M3, MountingHole:MountingHole_3.2mm_M3
- C1, C2: value 0.1uF -> 100nF
- U1: value MPU-6050 -> LSM6DS3; footprint Sensor_Motion:InvenSense_QFN-24_4x4mm_P0.5mm -> Package_LGA:LGA-14_3x2.5mm_P0.5mm_LayoutBorder3x4y
- moved C1 9.78 mm to (166.4, 88.9)
- moved C2 5.35 mm to (166.3, 91.4), turned to 0 degrees
- moved U1 3.62 mm to (163.4, 90.9), turned to 90 degrees
- renumbered GND1 to U2
Connections:
- C1 pad 1: Net-(U1-REGOUT) -> /3V3
- R2 pad 1: Net-(GND1-GPIO21) -> /SCL
- R3 pad 1: Net-(GND1-GPIO20) -> /I2CSDA
- U1 pad 10: Net-(U1-REGOUT) -> unconnected-(U1-NC-Pad10)
- U1 pad 11: GND -> unconnected-(U1-NC-Pad11)
- U1 pad 12: unconnected-(U1-INT-Pad12) -> /3V3
- U1 pad 13: /3V3 -> /SCL
- U1 pad 14: unconnected-(U1-NC-Pad14) -> /I2CSDA
- U1 pad 2: unconnected-(U1-NC-Pad2) -> GND
- U1 pad 3: unconnected-(U1-NC-Pad3) -> GND
- U1 pad 5: unconnected-(U1-NC-Pad5) -> /3V3
- U1 pad 6: unconnected-(U1-AUX_DA-Pad6) -> GND
- U1 pad 7: unconnected-(U1-AUX_CL-Pad7) -> GND
- U1 pad 9: GND -> unconnected-(U1-INT2-Pad9)
- U2 pad 26: Net-(GND1-GPIO20) -> /I2CSDA
- U2 pad 27: Net-(GND1-GPIO21) -> /SCL
Routing:
- net /3V3: track 132.2 -> 154.3 mm
- net /I2CSDA: track 0.00 -> 16.7 mm
- net Net-(GND1-GPIO21): track 16.5 -> 0.00 mm
- net Net-(GND1-GPIO20): track 16.3 -> 0.00 mm
- net /SCL: track 0.00 -> 15.8 mm
- net Net-(U1-CPOUT): track 3.56 -> 0.00 mm
- net Net-(U1-REGOUT): track 2.14 -> 0.00 mm
- net GND: track 22.2 -> 23.7 mm, vias 10 -> 9
Other:
- board text added: "PCB rev 2.2.2"
- board text removed: "PCB rev 2.1.0"
