File: design/design.kicad_sch (KiCad schematic)
At the start: 26 parts, among them J2 Conn_01x08_Socket, SW1 SW_Push, SW10 SW_Push, SW11 SW_Push, SW12 SW_Push, SW13 SW_Push, SW2 SW_Push, SW3 SW_Push, SW4 SW_Push, SW5 SW_Push, SW6 SW_Push, SW7 SW_Push, SW8 SW_Push, SW9 SW_Push, U1 MPU-6050

Commit message: Version using LSM6DS3 (C967633) chip
Parts:
- removed C1, C2: 0.1uF, Capacitor_SMD:C_0402_1005Metric, symbol Device:C
- removed C3: 2.2nF, Capacitor_SMD:C_0603_1608Metric, symbol Device:C
- removed C4: 10nF, Capacitor_SMD:C_0603_1608Metric, symbol Device:C
- removed U1: MPU-6050, Sensor_Motion:InvenSense_QFN-24_4x4mm_P0.5mm, symbol Sensor_Motion:MPU-6050
- added C1, C2: 100nF, Capacitor_SMD:C_0402_1005Metric, symbol Device:C_Small
- added U1: LSM6DS3, Package_LGA:LGA-14_3x2.5mm_P0.5mm_LayoutBorder3x4y, symbol Sensor_Motion:LSM6DS3
- renumbered GND1 to U2
Connections:
- net 3V3: now also C1.1, C2.1, U1.12 (CS), U1.5 (VDDIO), U1.8 (VDD)
- net GND: now also C1.2, C2.2, U1.1 (SDO/SA0), U1.2 (SDX), U1.3 (SCX), U1.6 (GND), U1.7 (GND)
- net SCL: now reaches R2.1, U2.27 (GPIO21)
- net SCL: now also U1.13 (SCL)
- net I2CSDA: now reaches R3.1, U2.26 (GPIO20)
- net I2CSDA: now also U1.14 (SDA)

Commit message: Redesigned to use clone accelerometer module
Parts:
- removed U1: LSM6DS3, Package_LGA:LGA-14_3x2.5mm_P0.5mm_LayoutBorder3x4y, symbol Sensor_Motion:LSM6DS3
- added U2: LIS2DW12, LIS2DW12:LGA12R50P4X4_200X200X70, symbol LIS2DW12:LIS2DW12
- renumbered U2 to U1
Connections:
- net 3V3: now also U2.10 (VDD_IO), U2.2 (CS), U2.9 (VDD)
- net GND: now also U2.3 (SDO/SDA0), U2.6 (GND), U2.7 (RES), U2.8 (GND)
- net I2CSDA: now also U2.4 (SDA/SDI/SDO)
- net SCL: now also U2.1 (SCL/SPC)
- no-connect marks 7 -> 9
