File: design/old/pcb_old.kicad_pcb (KiCad board)
At the start: 2 copper layers, 176.5 x 83.2 mm, 24 parts, among them J2 Conn_01x08_Socket, SW1 SW_Push, SW10 SW_Push, SW11 SW_Push, SW12 SW_Push, SW13 SW_Push, SW2 SW_Push, SW3 SW_Push, SW4 SW_Push, SW5 SW_Push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

Commit message: Improved poster and renders, re-exported gerber file
Changed lines of the file:
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@@
+	)
+	(gr_line
+		(start 66 58.75)
+		(end 66 58.5)
+		(stroke
+			(width 0.2)
+			(type default)
+		)
+		(layer "F.Cu")
+	)
+	(gr_line
+		(start 66 69.75)
+		(end 66 58.75)
+		(stroke
+			(width 0.2)
+			(type default)
+		)
+		(layer "F.Cu")
+	)
+	(gr_line
+		(start 76.75 58.5)
+		(end 66 58.5)
+		(stroke
+			(width 0.2)
+			(type default)
+		)
+		(layer "F.Cu")
+	)
+	(gr_line
+		(start 232.5 58.5)
+		(end 246.75 58.5)
+		(stroke
+			(width 0.2)
+			(type default)
+		)
+		(layer "F.Cu")
+	)
+	(gr_line
+		(start 242.5 73.75)
+		(end 242.5 58.5)
+		(stroke
+			(width 0.2)
+			(type default)
+		)
+		(layer "F.Cu")
 	)
 	(gr_line
